File: test-jig/layout/test-jig.kicad_pcb (KiCad board)
At the start: 2 copper layers, 100 x 100 mm, 40 parts, among them J1 Conn_02x05_Odd_Even, J2 Conn_02x10_Odd_Even, J3 Conn_02x05_Odd_Even

Commit message: test-jig: route the traces
Parts:
- added REF**: Toggle_Clamp_GH13009, footprints:Toggle_Clamp_GH13009, F.Cu at (159.3, 78.0)
- moved REF** 4.42 mm to (181.5, 72.5)
- moved REF** 3.89 mm to (170.5, 71.8)
Routing:
- net GND: track 0.00 -> 133.5 mm
- net DBG_SWO: track 0.00 -> 105.3 mm
- net DBG_SWCLK: track 0.00 -> 104.8 mm
- net VDD: track 0.00 -> 104.4 mm
- net DBG_SWDIO: track 0.00 -> 104.2 mm
- net RESET: track 0.00 -> 100.1 mm
- net ETM_TD0: track 0.00 -> 90.7 mm
- net ETM_TCLK: track 0.00 -> 87.3 mm
- net USART_TX: track 0.00 -> 83.7 mm
- net USART_RX: track 0.00 -> 81.2 mm
Other:
- net class Default: clearance 0.2 -> 0.1524; trace_width 0.25 -> 0.1524
- rule trace_clearance: 0.2 -> 0.1524
- rule trace_min: 0.2 -> 0.1524
- board text added: "JLCJLCJLCJLC"
- board text added: "clever-card test jig v0.1"
